File: firstPCB/lightSensitiveAlarm/lightSensitiveAlarm.kicad_sch (KiCad schematic)
At the start: 6 parts, among them Q1 BC547

Commit message: mmmmmhm
Connections:
- net VCC: now reaches BT1.1 (+), BZ1.1 (-), C1.1, R1.1
- net Ground: now reaches BT1.2 (-), Q1.3 (E), R2.2
Changed lines of the file:
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@@
     (stroke (width 0) (type default))
+  )
+  (label "Ground" (at 135.89 102.87 0) (fields_autoplaced)
+    (effects (font (size 1.27 1.27)) (justify left bottom))
+  )
+  (label "VCC" (at 132.08 88.9 0) (fields_autoplaced)
+    (effects (font (size 1.27 1.27)) (justify left bottom))
   )
   (symbol (lib_id "Device:Battery") (at 132.08 95.25 0) (unit 1)
